File: Hardware/Production/Qwiic_RFID_Tag-Panel.brd (EAGLE design)
At the start: 30.5 x 44.5 mm, 50 parts, among them J1 Qwiic, J2 Qwiic, U1 ST25DV64KC

Commit message: Created production files
Parts:
- added C10, C12, C4, C6, C8: 0.1uF, SparkFun-Capacitors:0603
- added C11, C3, C5, C7, C9: 4.7pF, SparkFun-Capacitors:0603
- added D2, D3, D4, D5, D6: RED, SparkFun-LED:LED-0603
- added E$1, E$2, E$3, E$4: (no value), SparkFun-Aesthetics:FIDUCIAL-1X2
- added E$5, E$6: (no value), SparkFun-Retired:FIDUCIAL-1.5X3
- added FD10, FD11, FD12, FD13, FD14, FD15, FD16, FD17, FD18, FD19, FD20, FD21, FD22, FD23, FD24, FD5, FD6, FD7, FD8, FD9: FIDUCIAL1X2, SparkFun-Aesthetics:FIDUCIAL-1X2
- added FRAME2, FRAME3, FRAME4, FRAME5, FRAME6: FRAME-LETTERNO_PACKAGE, SparkFun-Aesthetics:DUMMY
- added H10, H11, H12, H13, H14, H15, H16, H17, H18, H19, H20, H21, H22, H23, H24, H5, H6, H7, H8, H9: STAND-OFF, SparkFun-Hardware:STAND-OFF
- added J10, J11, J13, J14, J16, J17, J4, J5, J7, J8: Qwiic, SparkFun-Connectors:JST04_1MM_RA
- added J12, J15, J18, J6, J9: (no value), SparkFun-Connectors:1X06_NO_SILK
- added JP10, JP13, JP16, JP4, JP7: JUMPER-SMT_3_2-NC_TRACE_SILK, SparkFun-Jumpers:SMT-JUMPER_3_2-NC_TRACE_SILK
- added JP11, JP12, JP14, JP15, JP17, JP18, JP5, JP6, JP8, JP9: JUMPER-SMT_2_NC_TRACE_SILK, SparkFun-Jumpers:SMT-JUMPER_2_NC_TRACE_SILK
- added L2, L3, L4, L5, L6: PCB_4UH_INDUCTOR, SparkFun-Coils:PCB_4UH_INDUCTOR
- added LOGO10, LOGO13, LOGO16, LOGO4, LOGO7: OSHW-LOGOMINI, SparkFun-Aesthetics:OSHW-LOGO-MINI
- added LOGO11, LOGO12, LOGO14, LOGO15, LOGO17, LOGO18, LOGO5, LOGO6, LOGO8, LOGO9: QWIIC_LOGO_4MM, SparkFun-Aesthetics:QWIIC_4MM
- added R10, R13, R14, R17, R18, R21, R22, R5, R6, R9: 2.2k, SparkFun-Resistors:0603
- added R11, R15, R19, R23, R7: 1k, SparkFun-Resistors:0603
- added R12, R16, R20, R24, R8: 10k, SparkFun-Resistors:0603
- added U$100, U$111, U$123, U$134, U$31, U$42, U$54, U$65, U$77, U$88: (no value), output:#VEH#7
- added U$101, U$124, U$32, U$55, U$78: (no value), output:PWR11
- added U$102, U$125, U$33, U$56, U$79: (no value), output:MADE_IN_THE_USA27
- added U$103, U$126, U$34, U$57, U$80: (no value), output:#I2C#11
- added U$104, U$127, U$35, U$58, U$81: (no value), output:##GPO##9
- added U$105, U$128, U$36, U$59, U$82: (no value), output:#LED#10
- added U$106, U$119, U$129, U$27, U$37, U$50, U$60, U$73, U$83, U$96: (no value), output:#GND#4
- added U$107, U$118, U$130, U$26, U$38, U$49, U$61, U$72, U$84, U$95: (no value), output:#3#3V#0
- added U$108, U$120, U$131, U$28, U$39, U$51, U$62, U$74, U$85, U$97: (no value), output:#SDA#5
- added U$109, U$121, U$132, U$29, U$40, U$52, U$63, U$75, U$86, U$98: (no value), output:#SCL#6
- added U$110, U$122, U$133, U$30, U$41, U$53, U$64, U$76, U$87, U$99: (no value), output:##GPO##8
- added U$112, U$115, U$135, U$138, U$43, U$46, U$66, U$69, U$89, U$92: (no value), output:QWIIC12
- added U$113, U$114, U$136, U$137, U$44, U$45, U$67, U$68, U$90, U$91: (no value), output:RFID_TAG13
- added U$116, U$117, U$24, U$25, U$47, U$48, U$70, U$71, U$93, U$94: SPARKX-LOGO5, SparkX:SPARKX-LARGE
- added U2, U3, U4, U5, U6: ST25DV64KC, SparkFun-RF:SO08
Connections:
- new net !GPO!1: J6.5, R8.1, U2.7
- new net !GPO!2: J9.5, R12.1, U3.7
- new net !GPO!3: J12.5, R16.1, U4.7
- new net !GPO!4: J15.5, R20.1, U5.7
- new net !GPO!5: J18.5, R24.1, U6.7
- new net 3.3V1: C4.1, J4.2, J5.2, J6.2, JP4.2, JP5.2, JP6.2, U2.8
- new net 3.3V2: C6.1, J7.2, J8.2, J9.2, JP7.2, JP8.2, JP9.2, U3.8
- new net 3.3V3: C8.1, J10.2, J11.2, J12.2, JP10.2, JP11.2, JP12.2, U4.8
- new net 3.3V4: C10.1, J13.2, J14.2, J15.2, JP13.2, JP14.2, JP15.2, U5.8
- new net 3.3V5: C12.1, J16.2, J17.2, J18.2, JP16.2, JP17.2, JP18.2, U6.8
- new net AC10: C11.2, L6.IN1, U6.2
- new net AC11: C11.1, L6.IN2, U6.3
- new net AC2: C3.2, L2.IN1, U2.2
- new net AC3: C3.1, L2.IN2, U2.3
- new net AC4: C5.2, L3.IN1, U3.2
- new net AC5: C5.1, L3.IN2, U3.3
- new net AC6: C7.2, L4.IN1, U4.2
- new net AC7: C7.1, L4.IN2, U4.3
- new net AC8: C9.2, L5.IN1, U5.2
- new net AC9: C9.1, L5.IN2, U5.3
- new net GND1: C4.2, D2.C, J4.1, J5.1, J6.1, U2.4
- new net GND2: C6.2, D3.C, J7.1, J8.1, J9.1, U3.4
- new net GND3: C8.2, D4.C, J10.1, J11.1, J12.1, U4.4
- new net GND4: C10.2, D5.C, J13.1, J14.1, J15.1, U5.4
- new net GND5: C12.2, D6.C, J16.1, J17.1, J18.1, U6.4
- new net N$10: JP6.1, R8.2
- new net N$11: JP7.3, R9.2
- new net N$12: JP7.1, R10.2
- new net N$13: JP8.1, R11.2
- new net N$14: D3.A, R11.1
- new net N$15: JP9.1, R12.2
- new net N$16: JP10.3, R13.2
- new net N$17: JP10.1, R14.2
- new net N$18: JP11.1, R15.2
- new net N$19: D4.A, R15.1
- new net N$20: JP12.1, R16.2
- new net N$21: JP13.3, R17.2
- new net N$22: JP13.1, R18.2
- new net N$23: JP14.1, R19.2
- new net N$24: D5.A, R19.1
- new net N$25: JP15.1, R20.2
- new net N$26: JP16.3, R21.2
- new net N$27: JP16.1, R22.2
- new net N$28: JP17.1, R23.2
- new net N$29: D6.A, R23.1
- new net N$30: JP18.1, R24.2
- new net N$6: JP4.3, R5.2
- new net N$7: JP4.1, R6.2
- new net N$8: JP5.1, R7.2
- new net N$9: D2.A, R7.1
- new net SCL1: J4.4, J5.4, J6.4, R6.1, U2.6
- new net SCL2: J7.4, J8.4, J9.4, R10.1, U3.6
- new net SCL3: J10.4, J11.4, J12.4, R14.1, U4.6
- new net SCL4: J13.4, J14.4, J15.4, R18.1, U5.6
- new net SCL5: J16.4, J17.4, J18.4, R22.1, U6.6
- new net SDA1: J4.3, J5.3, J6.3, R5.1, U2.5
- new net SDA2: J7.3, J8.3, J9.3, R9.1, U3.5
- new net SDA3: J10.3, J11.3, J12.3, R13.1, U4.5
- new net SDA4: J13.3, J14.3, J15.3, R17.1, U5.5
- new net SDA5: J16.3, J17.3, J18.3, R21.1, U6.5
- new net VEH1: J6.6, U2.1
- new net VEH2: J9.6, U3.1
- new net VEH3: J12.6, U4.1
- new net VEH4: J15.6, U5.1
- new net VEH5: J18.6, U6.1
Routing:
- net 3.3V5: track 0.00 -> 48.7 mm, vias 0 -> 4
- net 3.3V4: track 0.00 -> 48.7 mm, vias 0 -> 4
- net 3.3V3: track 0.00 -> 48.7 mm, vias 0 -> 4
- net 3.3V1: track 0.00 -> 48.7 mm, vias 0 -> 4
- net 3.3V2: track 0.00 -> 48.7 mm, vias 0 -> 4
- net SDA5: track 0.00 -> 37.9 mm, vias 0 -> 2
- net SDA3: track 0.00 -> 37.9 mm, vias 0 -> 2
- net SDA4: track 0.00 -> 37.9 mm, vias 0 -> 2
- net SDA2: track 0.00 -> 37.9 mm, vias 0 -> 2
- net SDA1: track 0.00 -> 37.9 mm, vias 0 -> 2
- net SCL5: track 0.00 -> 33.1 mm, vias 0 -> 3
- net SCL3: track 0.00 -> 33.1 mm, vias 0 -> 3
- net SCL2: track 0.00 -> 33.1 mm, vias 0 -> 3
- net SCL1: track 0.00 -> 33.1 mm, vias 0 -> 3
- net SCL4: track 0.00 -> 33.1 mm, vias 0 -> 3
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- added copper zone on layer 1, net GND1
- added copper zone on layer 16, net GND1
- added copper zone on layer 1, net GND2
- added copper zone on layer 16, net GND2
- added copper zone on layer 1, net GND3
- added copper zone on layer 16, net GND3
- added copper zone on layer 1, net GND4
- added copper zone on layer 16, net GND4
- added copper zone on layer 1, net GND5
- added copper zone on layer 16, net GND5
Other:
- board size 30.5 x 44.5 mm -> 114.5 x 105.6 mm
- board text added: "v-score"
- board text removed: "Dimensions in inches"

Commit message: Created PCB production files.
Parts:
- removed U$127: (no value), output:##GPO##9
- removed U$128: (no value), output:#LED#10
- removed U$129: (no value), output:#GND#4
- removed U$130: (no value), output:#3#3V#0
- removed U$131: (no value), output:#SDA#5
- removed U$132: (no value), output:#SCL#6
- removed U$133: (no value), output:##GPO##8
- removed U$134: (no value), output:#VEH#7
- removed U$135, U$138: (no value), output:QWIIC12
- removed U$136, U$137: (no value), output:RFID_TAG13
- LOGO11, LOGO12, LOGO14, LOGO15, LOGO17, LOGO18, LOGO2, LOGO3, LOGO5, LOGO6, LOGO8, LOGO9: value QWIIC_LOGO_4MM -> QWIIC_LOGO_7MM; device SparkFun-Aesthetics:QWIIC_4MM -> SparkFun-Aesthetics:QWIIC_7MM
- U$10, U$13, U$43: value (none) -> SPARKX-LOGO5; device output:QWIIC12 -> SparkX:SPARKX-LARGE
- U$100: device output:#VEH#7 -> output:#SDA#5
- U$101: device output:PWR11 -> output:#SCL#6
- U$102: device output:MADE_IN_THE_USA27 -> output:##GPO##8
- U$103: device output:#I2C#11 -> output:#VEH#7
- U$104: device output:##GPO##9 -> output:RFID_TAG13
- U$105: device output:#LED#10 -> output:RFID_TAG13
- U$106: value (none) -> SPARKX-LOGO5; device output:#GND#4 -> SparkX:SPARKX-LARGE
- U$107: value (none) -> SPARKX-LOGO5; device output:#3#3V#0 -> SparkX:SPARKX-LARGE
- U$108, U$120: device output:#SDA#5 -> output:#3#3V#0
- U$109, U$98: device output:#SCL#6 -> output:#GND#4
- U$110: device output:##GPO##8 -> output:#SDA#5
- U$111: device output:#VEH#7 -> output:#SCL#6
- U$112: device output:QWIIC12 -> output:##GPO##8
- U$113: device output:RFID_TAG13 -> output:#VEH#7
- U$114: device output:RFID_TAG13 -> output:PWR11
- U$115: device output:QWIIC12 -> output:MADE_IN_THE_USA27
- U$116: value SPARKX-LOGO5 -> (none); device SparkX:SPARKX-LARGE -> output:#I2C#11
- U$117: value SPARKX-LOGO5 -> (none); device SparkX:SPARKX-LARGE -> output:##GPO##9
- U$118: device output:#3#3V#0 -> output:#LED#10
- U$121: device output:#SCL#6 -> output:#SDA#5
- U$122: device output:##GPO##8 -> output:#SCL#6
- U$123: device output:#VEH#7 -> output:##GPO##8
- U$124: device output:PWR11 -> output:#VEH#7
- U$125: device output:MADE_IN_THE_USA27 -> output:RFID_TAG13
- U$126: device output:#I2C#11 -> output:RFID_TAG13
- U$24: value SPARKX-LOGO5 -> (none); device SparkX:SPARKX-LARGE -> output:#3#3V#0
- U$25: value SPARKX-LOGO5 -> (none); device SparkX:SPARKX-LARGE -> output:#GND#4
- U$26: device output:#3#3V#0 -> output:#SDA#5
- U$27: device output:#GND#4 -> output:#SCL#6
- U$28, U$39: device output:#SDA#5 -> output:##GPO##8
- U$29, U$40: device output:#SCL#6 -> output:#VEH#7
- U$30: device output:##GPO##8 -> output:PWR11
- U$31: device output:#VEH#7 -> output:MADE_IN_THE_USA27
- U$32: device output:PWR11 -> output:#I2C#11
- U$33: device output:MADE_IN_THE_USA27 -> output:##GPO##9
- U$34: device output:#I2C#11 -> output:#LED#10
- U$35: device output:##GPO##9 -> output:#GND#4
- U$36: device output:#LED#10 -> output:#3#3V#0
- U$37: device output:#GND#4 -> output:#SDA#5
- U$38: device output:#3#3V#0 -> output:#SCL#6
- U$41: device output:##GPO##8 -> output:RFID_TAG13
- U$42: device output:#VEH#7 -> output:RFID_TAG13
- U$44: value (none) -> SPARKX-LOGO5; device output:RFID_TAG13 -> SparkX:SPARKX-LARGE
- U$45: device output:RFID_TAG13 -> output:#3#3V#0
- U$46: device output:QWIIC12 -> output:#GND#4
- U$47: value SPARKX-LOGO5 -> (none); device SparkX:SPARKX-LARGE -> output:#SDA#5
- U$48: value SPARKX-LOGO5 -> (none); device SparkX:SPARKX-LARGE -> output:#SCL#6
- U$49: device output:#3#3V#0 -> output:##GPO##8
- U$50: device output:#GND#4 -> output:#VEH#7
- U$51: device output:#SDA#5 -> output:PWR11
- U$52: device output:#SCL#6 -> output:MADE_IN_THE_USA27
- U$53: device output:##GPO##8 -> output:#I2C#11
- U$54: device output:#VEH#7 -> output:##GPO##9
- U$55: device output:PWR11 -> output:#LED#10
- U$56: device output:MADE_IN_THE_USA27 -> output:#GND#4
- U$57: device output:#I2C#11 -> output:#3#3V#0
- U$58: device output:##GPO##9 -> output:#SDA#5
- U$59: device output:#LED#10 -> output:#SCL#6
- U$60: device output:#GND#4 -> output:##GPO##8
- U$61: device output:#3#3V#0 -> output:#VEH#7
- U$62: device output:#SDA#5 -> output:RFID_TAG13
- U$63: device output:#SCL#6 -> output:RFID_TAG13
- U$64: value (none) -> SPARKX-LOGO5; device output:##GPO##8 -> SparkX:SPARKX-LARGE
- U$65: value (none) -> SPARKX-LOGO5; device output:#VEH#7 -> SparkX:SPARKX-LARGE
- U$66: device output:QWIIC12 -> output:#3#3V#0
- U$67: device output:RFID_TAG13 -> output:#GND#4
- U$68: device output:RFID_TAG13 -> output:#SDA#5
- U$69: device output:QWIIC12 -> output:#SCL#6
- U$70: value SPARKX-LOGO5 -> (none); device SparkX:SPARKX-LARGE -> output:##GPO##8
- U$71: value SPARKX-LOGO5 -> (none); device SparkX:SPARKX-LARGE -> output:#VEH#7
- U$72: device output:#3#3V#0 -> output:PWR11
- U$73: device output:#GND#4 -> output:MADE_IN_THE_USA27
- U$74: device output:#SDA#5 -> output:#I2C#11
- U$75: device output:#SCL#6 -> output:##GPO##9
- U$76: device output:##GPO##8 -> output:#LED#10
- U$77, U$88: device output:#VEH#7 -> output:#GND#4
- U$78: device output:PWR11 -> output:#3#3V#0
- U$79: device output:MADE_IN_THE_USA27 -> output:#SDA#5
- U$80: device output:#I2C#11 -> output:#SCL#6
- U$81: device output:##GPO##9 -> output:##GPO##8
- U$82: device output:#LED#10 -> output:#VEH#7
- U$83: device output:#GND#4 -> output:RFID_TAG13
- U$84: device output:#3#3V#0 -> output:RFID_TAG13
- U$85: value (none) -> SPARKX-LOGO5; device output:#SDA#5 -> SparkX:SPARKX-LARGE
- U$86: value (none) -> SPARKX-LOGO5; device output:#SCL#6 -> SparkX:SPARKX-LARGE
- U$87, U$99: device output:##GPO##8 -> output:#3#3V#0
- U$89: device output:QWIIC12 -> output:#SDA#5
- U$90: device output:RFID_TAG13 -> output:#SCL#6
- U$91: device output:RFID_TAG13 -> output:##GPO##8
- U$92: device output:QWIIC12 -> output:#VEH#7
- U$93: value SPARKX-LOGO5 -> (none); device SparkX:SPARKX-LARGE -> output:PWR11
- U$94: value SPARKX-LOGO5 -> (none); device SparkX:SPARKX-LARGE -> output:MADE_IN_THE_USA27
- U$95: device output:#3#3V#0 -> output:#I2C#11
- U$96: device output:#GND#4 -> output:##GPO##9
- U$97: device output:#SDA#5 -> output:#LED#10
- moved U$65 109.7 mm to (15.2, 86.9), turned to 0 degrees
- moved U$64 98.5 mm to (15.2, 74.2), flipped to the top, turned to 0 degrees
- moved U$67 69.6 mm to (8.89, 46.7), turned to 90 degrees
- moved U$66 66.9 mm to (11.4, 46.7), turned to 90 degrees
- moved U$68 66.4 mm to (14.0, 46.7), flipped to the top, turned to 90 degrees
- moved U$69 63.4 mm to (16.5, 46.7), flipped to the top, turned to 90 degrees
- moved U$112 54.1 mm to (81.0, 46.7), turned to 90 degrees
- moved U$113 53.9 mm to (83.6, 46.7), turned to 90 degrees
- moved U$107 52.4 mm to (77.2, 86.9), turned to 0 degrees
- moved U$89 51.4 mm to (45.0, 46.7), turned to 90 degrees
- moved U$90 50.9 mm to (47.5, 46.7), turned to 90 degrees
- moved U$86 49.5 mm to (46.2, 86.9), turned to 0 degrees
- moved U$92 48.4 mm to (52.6, 46.7), flipped to the top, turned to 90 degrees
- moved U$106 45.6 mm to (77.2, 74.2), flipped to the top, turned to 0 degrees
- moved U$91 45.1 mm to (50.0, 46.7), flipped to the top, turned to 90 degrees
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Other:
- board size 114.5 x 105.6 mm -> 112.5 x 103.6 mm
