File: Hardware/Production/Qwiic_RFID_Tag-Panel.brd (EAGLE design)
At the start: 112.5 x 103.6 mm, 306 parts, among them J1 Qwiic, J10 Qwiic, J11 Qwiic, J13 Qwiic, J14 Qwiic, J16 Qwiic, J17 Qwiic, J2 Qwiic, J4 Qwiic, J5 Qwiic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

Commit message: X02 PCB
Parts:
- removed LOGO13, LOGO16: OSHW-LOGOMINI, SparkFun-Aesthetics:OSHW-LOGO-MINI
- removed LOGO14, LOGO15, LOGO17, LOGO18: QWIIC_LOGO_7MM, SparkFun-Aesthetics:QWIIC_7MM
- removed U$133: (no value), output:#VEH#7
- removed U$134, U$135: (no value), output:RFID_TAG13
- removed U$136, U$137: (no value), SER:ST25DV64KC5984
- removed U$138: (no value), output:MADE_IN_THE_USA20
- LOGO10, LOGO4: value OSHW-LOGOMINI -> QWIIC_LOGO_7MM; device SparkFun-Aesthetics:OSHW-LOGO-MINI -> SparkFun-Aesthetics:QWIIC_7MM
- LOGO11, LOGO2, LOGO5, LOGO9: value QWIIC_LOGO_7MM -> OSHW-LOGOMINI; device SparkFun-Aesthetics:QWIIC_7MM -> SparkFun-Aesthetics:OSHW-LOGO-MINI
- U$10: value SPARKX-LOGO5 -> (none); device SparkX:SPARKX-LARGE -> output:DYNAMIC_RFID_TAG0
- U$100: device output:#VEH#7 -> output:#LED#10
- U$101: device output:PWR11 -> output:#GND#4
- U$102: device output:#I2C#11 -> output:#3#3V#0
- U$103: device output:##GPO##9 -> output:#SDA#5
- U$104: device output:#LED#10 -> output:#SCL#6
- U$105, U$73: device output:#GND#4 -> output:##GPO##8
- U$106, U$118: device output:#3#3V#0 -> output:#VEH#7
- U$107, U$130: device output:#SDA#5 -> SER:ST25DV64KC5984
- U$108, U$85: device output:#SCL#6 -> SER:ST25DV64KC5984
- U$109, U$132: device output:##GPO##8 -> output:DYNAMIC_RFID_TAG0
- U$11, U$43, U$65, U$66, U$88: device output:RFID_TAG13 -> output:DYNAMIC_RFID_TAG0
- U$110, U$87: device output:#VEH#7 -> output:DYNAMIC_RFID_TAG0
- U$111, U$112, U$12, U$89: value (none) -> SPARKX-LOGO5; device output:RFID_TAG13 -> SparkX:SPARKX-LARGE
- U$113, U$91: device SER:ST25DV64KC5984 -> output:#3#3V#0
- U$114: device SER:ST25DV64KC5984 -> output:#GND#4
- U$115: device output:MADE_IN_THE_USA20 -> output:#SDA#5
- U$116, U$94: value SPARKX-LOGO5 -> (none); device SparkX:SPARKX-LARGE -> output:#SCL#6
- U$117: value SPARKX-LOGO5 -> (none); device SparkX:SPARKX-LARGE -> output:##GPO##8
- U$119: device output:#GND#4 -> output:PWR11
- U$120: device output:#SDA#5 -> output:#I2C#11
- U$121: device output:#SCL#6 -> output:##GPO##9
- U$122: device output:##GPO##8 -> output:#LED#10
- U$123: device output:#VEH#7 -> output:#GND#4
- U$124: device output:PWR11 -> output:#3#3V#0
- U$125: device output:#I2C#11 -> output:#SDA#5
- U$126: device output:##GPO##9 -> output:#SCL#6
- U$127: device output:#LED#10 -> output:##GPO##8
- U$128, U$96: device output:#GND#4 -> output:#VEH#7
- U$129: device output:#3#3V#0 -> SER:ST25DV64KC5984
- U$131: device output:#SCL#6 -> output:DYNAMIC_RFID_TAG0
- U$34: device output:MADE_IN_THE_USA20 -> output:#LED#10
- U$35: device output:#LED#10 -> output:#GND#4
- U$36: device output:#GND#4 -> output:#3#3V#0
- U$37, U$49: device output:#3#3V#0 -> output:#SDA#5
- U$38: device output:#SDA#5 -> output:#SCL#6
- U$39: device output:#SCL#6 -> output:##GPO##8
- U$40: device output:##GPO##8 -> output:#VEH#7
- U$41, U$64: device output:#VEH#7 -> SER:ST25DV64KC5984
- U$42: device output:RFID_TAG13 -> SER:ST25DV64KC5984
- U$44: device SER:ST25DV64KC5984 -> output:DYNAMIC_RFID_TAG0
- U$45, U$67, U$68, U$90: value (none) -> SPARKX-LOGO5; device SER:ST25DV64KC5984 -> SparkX:SPARKX-LARGE
- U$46: value (none) -> SPARKX-LOGO5; device output:MADE_IN_THE_USA20 -> SparkX:SPARKX-LARGE
- U$47: value SPARKX-LOGO5 -> (none); device SparkX:SPARKX-LARGE -> output:#3#3V#0
- U$48, U$70: value SPARKX-LOGO5 -> (none); device SparkX:SPARKX-LARGE -> output:#GND#4
- U$50, U$82: device output:#GND#4 -> output:#SCL#6
- U$51, U$61: device output:#SDA#5 -> output:##GPO##8
- U$52, U$62: device output:#SCL#6 -> output:#VEH#7
- U$53: device output:##GPO##8 -> output:PWR11
- U$54: device output:#VEH#7 -> output:#I2C#11
- U$55: device output:PWR11 -> output:##GPO##9
- U$56: device output:#I2C#11 -> output:#LED#10
- U$57: device output:##GPO##9 -> output:#GND#4
- U$58: device output:#LED#10 -> output:#3#3V#0
- U$59: device output:#GND#4 -> output:#SDA#5
- U$60, U$72: device output:#3#3V#0 -> output:#SCL#6
- U$63, U$86: device output:##GPO##8 -> SER:ST25DV64KC5984
- U$69: device output:MADE_IN_THE_USA20 -> output:#3#3V#0
- U$71, U$93: value SPARKX-LOGO5 -> (none); device SparkX:SPARKX-LARGE -> output:#SDA#5
- U$74, U$84: device output:#SDA#5 -> output:#VEH#7
- U$75: device output:#SCL#6 -> output:PWR11
- U$76: device output:##GPO##8 -> output:#I2C#11
- U$77: device output:#VEH#7 -> output:##GPO##9
- U$78: device output:PWR11 -> output:#LED#10
- U$79: device output:#I2C#11 -> output:#GND#4
- U$80: device output:##GPO##9 -> output:#3#3V#0
- U$81: device output:#LED#10 -> output:#SDA#5
- U$83, U$95: device output:#3#3V#0 -> output:##GPO##8
- U$92: device output:MADE_IN_THE_USA20 -> output:#GND#4
- U$97: device output:#SDA#5 -> output:PWR11
- U$98: device output:#SCL#6 -> output:#I2C#11
- U$99: device output:##GPO##8 -> output:##GPO##9
- moved LOGO8 78.9 mm to (3.81, 60.2)
- moved LOGO11 77.1 mm to (90.7, 60.2), flipped to the bottom
- moved LOGO7 76.6 mm to (28.7, 60.2)
- moved U$67 69.5 mm to (15.2, 74.2)
- moved U$68 69.5 mm to (15.2, 74.2)
- moved U$69 62.1 mm to (11.4, 46.7), flipped to the top
- moved LOGO12 53.1 mm to (65.8, 60.2), flipped to the top
- moved U$34 51.5 mm to (52.2, 10.2), turned to 0 degrees
- moved U$113 49.1 mm to (73.4, 46.7), turned to 90 degrees
- moved U$91 49.1 mm to (42.4, 46.7), flipped to the top, turned to 90 degrees
- moved U$46 48.7 mm to (77.2, 29.2), turned to 0 degrees
- moved U$114 47.7 mm to (70.9, 46.7), flipped to the top, turned to 90 degrees
- moved LOGO2 47.4 mm to (59.7, 15.2)
- moved LOGO5 47.3 mm to (90.7, 15.2), flipped to the bottom
- moved U$115 45.3 mm to (75.9, 46.7), flipped to the top
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Other:
- board text added: "X02"
- board text removed: "X01"
