File: Hardware/Qwiic_RFID_Tag.brd (EAGLE design)
At the start: 30.5 x 44.5 mm, 50 parts, among them J1 Qwiic, J2 Qwiic, U1 ST25DV64KC

Commit message: X02 PCB
Parts:
- removed LOGO2: QWIIC_LOGO_7MM, SparkFun-Aesthetics:QWIIC_7MM
- removed U$12: (no value), output:RFID_TAG13
- removed U$34: (no value), output:MADE_IN_THE_USA20
- added U$10: (no value), output:DYNAMIC_RFID_TAG0
- U$11: device output:RFID_TAG13 -> output:DYNAMIC_RFID_TAG0
- moved LOGO3 19.8 mm to (3.81, 15.2)
- moved U$1 1.02 mm to (15.2, 29.2)
- moved U$2 0.76 mm to (15.2, 29.2)
- moved U$15 0.13 mm to (10.2, 12.6)
- moved U$16 0.13 mm to (21.2, 7.62)
- moved U$17 0.13 mm to (21.2, 10.2)
- flipped U$11 to the bottom
Other:
- board text added: "X02"
- board text removed: "X01"
